File: hardware/PCB/eagle/boards/sensor boards/fibre_sensor/fibre_sensor_board.brd (EAGLE design)
At the start: 14.9 x 12.7 mm, 7 parts

Commit message: updated
Parts:
- C1: device SparkFun-Capacitors:CAP-PTH-SMALL -> passive_components:TH_0.1-CAP
- D1: device SparkFun-LED:LTE-302 -> passive_components:TH_0.1-LED
- D2: device SparkFun-LED:LTE-302 -> passive_components:TH_0.1-PD
- JP1, JP2: device SparkFun-Connectors:1X04 -> passive_components:1X04
- R1, R2: device SparkFun-Resistors:AXIAL-0.3 -> passive_components:TH_0.3-RES
- moved JP1 3.81 mm to (2.54, 6.35), flipped to the bottom
- moved JP2 3.81 mm to (12.7, 6.35), flipped to the bottom
- flipped C1 to the bottom
Routing:
- net VCC: vias 0 -> 1
- net OAO: vias 0 -> 2
- net OA-: vias 0 -> 4
- net LED-: vias 0 -> 1
Changed lines of the file:
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@@
 <setting verticaltext="up"/>
 </settings>
-<grid distance="0.05" unitdist="inch" unit="inch" style="lines" multiple="1" display="yes" altdistance="0.025" altunitdist="inch" altunit="inch"/>
+<grid distance="0.05" unitdist="inch" unit="mm" style="lines" multiple="1" display="yes" altdistance="0.025" altunitdist="inch" altunit="inch"/>
 <layers>
-<layer number="1" name="Top" color="4" fill="1" visible="no" active="yes"/>
+<layer number="1" name="Top" color="4" fill="1" visible="yes" active="yes"/>
 <layer number="16" name="Bottom" color="1" fill="1" visible="yes" active="yes"/>
 <layer number="17" name="Pads" color="2" fill="1" visible="yes" active="yes"/>
@@
 </autorouter>
 <elements>
-<element name="JP1" library="SparkFun-Connectors" package="1X04" value="" x="2.54" y="10.16" rot="R270"/>
-<element name="JP2" library="SparkFun-Connectors" package="1X04" value="" x="12.7" y="10.16" rot="R270"/>
-<element name="R1" library="SparkFun-Resistors" package="AXIAL-0.3" value="1G" x="5.08" y="6.35" rot="R270"/>
-<element name="R2" library="SparkFun-Resistors" package="AXIAL-0.3" value="1G" x="7.62" y="6.35" rot="R90"/>
-<element name="C1" library="SparkFun-Capacitors" package="CAP-PTH-SMALL" value="" x="6.35" y="7.62" rot="R270"/>
-<element name="D1" library="SparkFun-LED" package="LTE-302" value="LED" x="10.16" y="8.89" rot="R90"/>
-<element name="D2" library="SparkFun-LED" package="LTE-302" value="PD" x="10.16" y="3.81" rot="R270"/>
+<element name="JP1" library="passive_components" package="1X04" value="" x="2.54" y="6.35" rot="MR270"/>
+<element name="JP2" library="passive_components" package="1X04" value="" x="12.7" y="6.35" rot="MR270"/>
+<element name="R1" library="passive_components" package="TH_0.3-RES" value="1G" x="5.08" y="6.35" rot="R270"/>
+<element name="R2" library="passive_components" package="TH_0.3-RES" value="1G" x="7.62" y="6.35" rot="R90"/>
+<element name="C1" library="passive_components" package="TH_0.1-CAP" value="" x="6.35" y="7.62" rot="MR270"/>
+<element name="D1" library="passive_components" package="TH_0.1-LED" value="LED" x="10.16" y="8.89" rot="R90"/>
+<element name="D2" library="passive_components" package="TH_0.1-PD" value="PD" x="10.16" y="3.81" rot="R270"/>
 </elements>
 <signals>
@@
 <wire x1="6.5" y1="5.25" x2="10" y2="5.25" width="0.25" layer="1"/>
 <wire x1="10" y1="5.25" x2="10.16" y2="5.08" width="0.25" layer="1"/>
-<wire x1="6.5" y1="5.25" x2="6.35" y2="5.08" width="0.25" layer="1"/>
+<wire x1="6.5" y1="5.25" x2="6.35" y2="5.08" width="0.25" layer="16"/>
 <wire x1="5" y1="10" x2="2.75" y2="7.75" width="0.25" layer="1"/>
-<wire x1="2.75" y1="7.75" x2="2.54" y2="7.62" width="0.25" layer="1"/>
+<wire x1="2.75" y1="7.75" x2="2.54" y2="7.62" width="0.25" layer="16"/>
 <wire x1="5" y1="10" x2="5.08" y2="10.16" width="0.25" layer="1"/>
 <wire x1="5" y1="5.25" x2="6.25" y2="5.25" width="0.25" layer="16"/>
 <wire x1="2.75" y1="7.5" x2="5" y2="5.25" width="0.25" layer="16"/>
-<wire x1="6.25" y1="5.25" x2="6.35" y2="5.08" width="0.25" layer="16"/>
-<wire x1="2.75" y1="7.5" x2="2.54" y2="7.62" width="0.25" layer="16"/>
+<wire x1="6.25" y1="5.25" x2="6.35" y2="5.08" width="0.25" layer="1"/>
+<wire x1="2.75" y1="7.5" x2="2.54" y2="7.62" width="0.25" layer="1"/>
+<via x="6.5" y="5.25" extent="1-16" drill="0.6" shape="square"/>
+<via x="6.25" y="5.25" extent="1-16" drill="0.6" shape="square"/>
+<via x="2.75" y="7.75" extent="1-16" drill="0.6" shape="square"/>
+<via x="2.75" y="7.5" extent="1-16" drill="0.6" shape="square"/>
 </signal>
 <signal name="OAO">
@@
 <wire x1="5" y1="5.5" x2="6.25" y2="6.75" width="0.25" layer="1"/>
 <wire x1="5" y1="2.75" x2="5" y2="5.5" width="0.25" layer="1"/>
-<wire x1="6.25" y1="7.5" x2="6.35" y2="7.62" width="0.25" layer="1"/>
+<wire x1="6.25" y1="7.5" x2="6.35" y2="7.62" width="0.25" layer="16"/>
 <wire x1="5" y1="2.75" x2="5.08" y2="2.54" width="0.25" layer="1"/>
 <wire x1="5" y1="2.5" x2="2.75" y2="2.5" width="0.25" layer="1"/>
-<wire x1="2.75" y1="2.5" x2="2.54" y2="2.54" width="0.25" layer="1"/>
+<wire x1="2.75" y1="2.5" x2="2.54" y2="2.54" width="0.25" layer="16"/>
 <wire x1="5" y1="2.5" x2="5.08" y2="2.54" width="0.25" layer="1"/>
+<via x="6.25" y="7.5" extent="1-16" drill="0.6" shape="square"/>
+<via x="2.75" y="2.5" extent="1-16" drill="0.6" shape="square"/>
 </signal>
 <signal name="VCC">
@@
 <wire x1="12.5" y1="10.25" x2="10.25" y2="10.25" width="0.25" layer="1"/>
 <wire x1="10.25" y1="10.25" x2="10.16" y2="10.16" width="0.25" layer="1"/>
-<wire x1="12.5" y1="10.25" x2="12.7" y2="10.16" width="0.25" layer="1"/>
+<wire x1="12.5" y1="10.25" x2="12.7" y2="10.16" width="0.25" layer="16"/>
+<via x="12.5" y="10.25" extent="1-16" drill="0.6" shape="square"/>
 </signal>
 <signal name="LED-">
@@
 <wire x1="12.5" y1="5" x2="11.5" y2="4" width="0.25" layer="1"/>
 <wire x1="7.75" y1="2.75" x2="7.62" y2="2.54" width="0.25" layer="1"/>
-<wire x1="12.5" y1="5" x2="12.7" y2="5.08" width="0.25" layer="1"/>
+<wire x1="12.5" y1="5" x2="12.7" y2="5.08" width="0.25" layer="16"/>
+<via x="12.5" y="5" extent="1-16" drill="0.6" shape="square"/>
 </signal>
 <signal name="N$1">
