File: hardware/PCB/eagle/boards/sensor boards/vbat/vbat_board.brd (EAGLE design)
At the start: 14.9 x 12.7 mm, 4 parts

Commit message: updated
Parts:
- JP1, JP2: device SparkFun-Connectors:1X04 -> passive_components:1X04
- R1, R2: device SparkFun-Resistors:AXIAL-0.3 -> passive_components:TH_0.3-RES
- moved JP1 3.81 mm to (2.54, 6.35), flipped to the bottom
- moved JP2 3.81 mm to (12.7, 6.35), flipped to the bottom
Routing:
- net VBAT/2: vias 0 -> 1
- net VBAT: vias 0 -> 1
- net GND: vias 0 -> 1
Changed lines of the file:
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@@
 <setting verticaltext="up"/>
 </settings>
-<grid distance="0.05" unitdist="inch" unit="inch" style="lines" multiple="1" display="yes" altdistance="0.025" altunitdist="inch" altunit="inch"/>
+<grid distance="0.05" unitdist="inch" unit="mm" style="lines" multiple="1" display="yes" altdistance="0.025" altunitdist="inch" altunit="inch"/>
 <layers>
 <layer number="1" name="Top" color="4" fill="1" visible="yes" active="yes"/>
@@
 <layer number="220" name="220bmp" color="21" fill="1" visible="no" active="no"/>
 <layer number="221" name="221bmp" color="22" fill="1" visible="no" active="no"/>
-<layer number="222" name="222bmp" color="23" fill="1" visible="no" active="no"/>
 <layer number="223" name="223bmp" color="24" fill="1" visible="no" active="no"/>
 <layer number="224" name="224bmp" color="25" fill="1" visible="no" active="no"/>
@@
 </autorouter>
 <elements>
-<element name="JP1" library="SparkFun-Connectors" package="1X04" value="" x="2.54" y="10.16" rot="R270"/>
-<element name="JP2" library="SparkFun-Connectors" package="1X04" value="" x="12.7" y="10.16" rot="R270"/>
-<element name="R1" library="SparkFun-Resistors" package="AXIAL-0.3" value="1G" x="8.89" y="6.35" rot="MR270"/>
-<element name="R2" library="SparkFun-Resistors" package="AXIAL-0.3" value="1G" x="6.35" y="6.35" rot="MR270"/>
+<element name="JP1" library="passive_components" package="1X04" value="" x="2.54" y="6.35" rot="MR270"/>
+<element name="JP2" library="passive_components" package="1X04" value="" x="12.7" y="6.35" rot="MR270"/>
+<element name="R1" library="passive_components" package="TH_0.3-RES" value="1G" x="8.89" y="6.35" rot="MR270"/>
+<element name="R2" library="passive_components" package="TH_0.3-RES" value="1G" x="6.35" y="6.35" rot="MR270"/>
 </elements>
 <signals>
@@
 <wire x1="12.5" y1="7.75" x2="11.25" y2="9" width="0.25" layer="1"/>
 <wire x1="6.5" y1="10.25" x2="6.35" y2="10.16" width="0.25" layer="1"/>
-<wire x1="12.5" y1="7.75" x2="12.7" y2="7.62" width="0.25" layer="1"/>
+<wire x1="12.5" y1="7.75" x2="12.7" y2="7.62" width="0.25" layer="16"/>
+<via x="12.5" y="7.75" extent="1-16" drill="0.6" shape="square"/>
 </signal>
 <signal name="VBAT/2">
@@
 <wire x1="12.5" y1="5" x2="9.25" y2="5" width="0.25" layer="1"/>
 <wire x1="6.5" y1="2.75" x2="6.35" y2="2.54" width="0.25" layer="1"/>
-<wire x1="12.5" y1="5" x2="12.7" y2="5.08" width="0.25" layer="1"/>
+<wire x1="12.5" y1="5" x2="12.7" y2="5.08" width="0.25" layer="16"/>
 <wire x1="9" y1="4.75" x2="9" y2="10" width="0.25" layer="1"/>
 <wire x1="9" y1="10" x2="8.89" y2="10.16" width="0.25" layer="1"/>
+<via x="12.5" y="5" extent="1-16" drill="0.6" shape="square"/>
 </signal>
 <signal name="VBAT">
@@
 <wire x1="12.5" y1="2.5" x2="9" y2="2.5" width="0.25" layer="1"/>
 <wire x1="9" y1="2.5" x2="8.89" y2="2.54" width="0.25" layer="1"/>
-<wire x1="12.5" y1="2.5" x2="12.7" y2="2.54" width="0.25" layer="1"/>
+<wire x1="12.5" y1="2.5" x2="12.7" y2="2.54" width="0.25" layer="16"/>
+<via x="12.5" y="2.5" extent="1-16" drill="0.6" shape="square"/>
 </signal>
 <signal name="N$1">
