File: hardware/PCB/eagle/boards/sensor boards/sensor_board/sensor_board.brd (EAGLE design)
At the start: 58.1 x 55.9 mm, 22 parts

Commit message: adjusted spacing on sensor board
- increased the spacing between components on the sensor board to aid
visibility of the values and names on the board
Parts:
- removed PWR_INT: (no value), passive_components:1X02
- added JP4: PWR_INT, passive_components:1X02
- JP3: value (none) -> PWR_EXT
- JP5: value (none) -> MCU1
- JP6: value (none) -> MCU2
- renumbered MCU1 to JP5, MCU2 to JP6, PWR_EXT to JP3
Connections:
- net VCC: now also JP4.1; no longer PWR_INT.1
- net VCC_INT: now also JP4.2; no longer PWR_INT.2
Routing:
- net VCC: track 103.8 -> 108.9 mm
- net VCC_INT: track 61.6 -> 60.1 mm
